Commit message: working on real robot

File: src/fmauch_universal_robot/ur_description/urdf/inc/ur5_cam_macro.xacro (robot description, xacro)
@@ -1,4 +1,4 @@
 <?xml version="1.0"?>
-<robot xmlns:xacro="http://wiki.ros.org/xacro">
+<robot xmlns:xacro="http://wiki.ros.org/xacro" name="ur5_cam">
   <xacro:macro name="ur5_cam" params="prefix">
     <!--

File: src/fmauch_universal_robot/ur_description/urdf/inc/ur5_light_bar_macro.xacro (robot description, xacro)
@@ -1,4 +1,4 @@
 <?xml version="1.0"?>
-<robot xmlns:xacro="http://wiki.ros.org/xacro">
+<robot xmlns:xacro="http://wiki.ros.org/xacro" name="ur5_light_bar">
   <xacro:macro name="ur5_light_bar" params="prefix">
     <xacro:include filename="$(find ur_description)/urdf/inc/ur5_macro.xacro" />

File: src/fmauch_universal_robot/ur_description/urdf/vision_application.xacro (robot description, xacro)
@@ -13,5 +13,5 @@
     <parent link="point_0" />
     <child link="ur5_cam_1_base_link" /> <!-- TODO: check base_link name of robot -->
-    <origin xyz="0 0.0 0" rpy="0.0 0.0 0.0" />
+    <origin xyz="0 0.0 0" rpy="0.0 0.0 -0.785398163" />
   </joint>
   <!-- define the ur5's position and orientation in the world coordinate system -->
@@ -19,5 +19,5 @@
     <parent link="point_0" />
     <child link="ur5_light_bar_1_base_link" /> <!-- TODO: check base_link name of robot -->
-    <origin xyz="1.1945 0.176 -0.07" rpy="0.0 0.0 0.0" />
+    <origin xyz="1.1945 0.176 -0.07" rpy="0.0 0.0 2.35619449" />
   </joint>
 </robot>
