Commit message: publish move goal via MoveIt + auto load scene

File: src/fmauch_universal_robot/ur_description/urdf/inc/b_and_r_cam_macro.xacro (robot description, xacro)
@@ -9,5 +9,5 @@
       <parent link="${connected_to}"/>
       <child link="${prefix}b_and_r_cam"/>
-      <!-- The tool is directly attached to the flange. -->
+      <!-- Tool position in relation to mount -->
       <origin rpy="-1.57079633 0 0" xyz="0.0 -0.063 -0.053"/>
     </joint>
@@ -28,5 +28,5 @@
         </geometry>
         <material>
-          <color rgba="0.8 0.7 0 1"/>
+          <color rgba="1 0.4 0 1"/>
         </material>
       </collision>

File: src/fmauch_universal_robot/ur_description/urdf/inc/b_and_r_light_bar_macro.xacro (robot description, xacro)
@@ -9,5 +9,5 @@
       <parent link="${connected_to}"/>
       <child link="${prefix}b_and_r_light_bar"/>
-      <!-- The tool is directly attached to the flange. -->
+      <!-- Tool position in relation to mount -->
       <origin rpy="-1.57079633 0 -1.57079633" xyz="0 -0.093 -0.049"/>
     </joint>
@@ -29,5 +29,5 @@
         </geometry>
         <material>
-          <color rgba="0.8 0.4 0"/>
+          <color rgba="1 0.4 0"/>
         </material>
       </collision>

File: src/fmauch_universal_robot/ur_description/urdf/inc/mount_macro.xacro (robot description, xacro)
@@ -9,5 +9,5 @@
       <parent link="${connected_to}" />
       <child link="${prefix}mount" />
-      <!-- The tool is directly attached to the flange. -->
+      <!-- The mount is posiontin in reltaion to the flange. -->
       <origin rpy="-1.57079633 0 -0.785398163" xyz="0 0 0" />
     </joint>

File: src/fmauch_universal_robot/ur_description/urdf/inc/ur5_cam_macro.xacro (robot description, xacro)
@@ -3,24 +3,14 @@
   <xacro:macro name="ur5_cam" params="prefix">
     <!--
-    This is a convenience top-level xacro which loads the macro for the UR5e
-    which defines the default values for the various "parameters files"
-    parameters for a UR5e.
-    This file is only useful when loading a stand-alone, completely isolated
-    robot with only default values for all parameters such as the kinematics,
-    visual and physical parameters and joint limits.
-    This file is not intended to be integrated into a larger scene or other
-    composite xacro.
-    Instead, xacro:include 'inc/ur5e_macro.xacro' and override the defaults
-    for the arguments to that macro.
-    Refer to 'inc/ur_macro.xacro' for more information.
+      Macro for creating an urdf file for an ur5 with a cam on it
   -->
     <xacro:include filename="$(find ur_description)/urdf/inc/ur5_macro.xacro" />
     <xacro:include filename="$(find ur_description)/urdf/inc/b_and_r_cam_macro.xacro" />
     <xacro:include filename="$(find ur_description)/urdf/inc/mount_macro.xacro" />
-    <!-- Specify name of robot -->
+    <!-- Use the macro for an ur5 robot and name it -->
     <xacro:ur5_robot prefix="${prefix}" />
-    <!-- Specify where the mount is connected to -->
+    <!-- Use the macro for a mount, Specify where the mount is connected to the ur5 -->
     <xacro:mount prefix="${prefix}" connected_to="${prefix}tool0" />
-    <!-- Specify where the camera is connected to and which robot it is mounted on -->
+    <!-- Use the macro for a camera, Specify where the camera is connected to the mount -->
     <xacro:b_and_r_cam prefix="${prefix}" connected_to="${prefix}mount" />
   </xacro:macro>

File: src/fmauch_universal_robot/ur_description/urdf/inc/ur5_light_bar_macro.xacro (robot description, xacro)
@@ -5,8 +5,9 @@
     <xacro:include filename="$(find ur_description)/urdf/inc/b_and_r_light_bar_macro.xacro" />
     <xacro:include filename="$(find ur_description)/urdf/inc/mount_macro.xacro" />
+    <!-- Use the macro for an ur5 robot and name it -->
     <xacro:ur5_robot prefix="${prefix}" />
-    <!-- Specify where the mount is connected to -->
+    <!-- Use the macro for a mount, Specify where the mount is connected to the ur5 -->
     <xacro:mount prefix="${prefix}" connected_to="${prefix}tool0" />
-    <!-- Specify where the camera is connected to -->
+    <!-- Use the macro for a light bar, Specify where the light bar is connected to the mount -->
     <xacro:b_and_r_light_bar prefix="${prefix}" connected_to="${prefix}mount" />
   </xacro:macro>

File: src/fmauch_universal_robot/ur_description/urdf/vision_application.xacro (robot description, xacro)
@@ -5,12 +5,12 @@
   <!-- define the ur5's position and orientation in the world coordinate system -->
   <!-- Specify name for ur5 with camera-->
-  <xacro:ur5_cam prefix="ur5_cam_1" />
+  <xacro:ur5_cam prefix="ur5_cam_1_" />
   <!-- Specify name for ur5 with light-->
-  <xacro:ur5_light_bar prefix="ur5_light_bar_1" />
+  <xacro:ur5_light_bar prefix="ur5_light_bar_1_" />
   <!-- define the ur5's position and orientation in the world coordinate system -->
   <link name="point_0" />
   <joint name="ur5_cam_1_point_0_joint" type="fixed">
     <parent link="point_0" />
-    <child link="ur5_cam_1base_link" /> <!-- TODO: check base_link name of robot -->
+    <child link="ur5_cam_1_base_link" /> <!-- TODO: check base_link name of robot -->
     <origin xyz="0 0.0 0" rpy="0.0 0.0 0.0" />
   </joint>
@@ -18,5 +18,5 @@
   <joint name="ur5_light_bar_1_point_0_joint" type="fixed">
     <parent link="point_0" />
-    <child link="ur5_light_bar_1base_link" /> <!-- TODO: check base_link name of robot -->
+    <child link="ur5_light_bar_1_base_link" /> <!-- TODO: check base_link name of robot -->
     <origin xyz="1.1945 0.176 -0.07" rpy="0.0 0.0 0.0" />
   </joint>

Commit message: Joint limits + look at viewpoint fixed

File: src/fmauch_universal_robot/ur_description/urdf/inc/b_and_r_cam_macro.xacro (robot description, xacro)
@@ -34,5 +34,5 @@
     <!-- TCP frame -->
     <joint name="${prefix}tcp_joint" type="fixed">
-      <origin rpy="-1.57079633 0 0" xyz="0.0 0.0 0.053" />
+      <origin rpy="-1.57079633 0 0" xyz="0.0 0.068 0.0" />
       <parent link="${prefix}b_and_r_cam"/>
       <child link="${prefix}tcp"/>

File: src/fmauch_universal_robot/ur_description/urdf/inc/b_and_r_light_bar_macro.xacro (robot description, xacro)
@@ -35,5 +35,5 @@
     <!-- TCP frame -->
     <joint name="${prefix}tcp_joint" type="fixed">
-      <origin rpy="-1.57079633 0 -1.57079633" xyz="0 0 0.049"/>
+      <origin rpy="-1.57079633 0 0" xyz="0 0.0862 0"/>
       <parent link="${prefix}b_and_r_light_bar"/>
       <child link="${prefix}tcp"/>

Commit message: collision free + look at point

File: src/fmauch_universal_robot/ur_description/urdf/inc/b_and_r_cam_macro.xacro (robot description, xacro)
@@ -34,5 +34,5 @@
     <!-- TCP frame -->
     <joint name="${prefix}tcp_joint" type="fixed">
-      <origin rpy="-1.57079633 0 0" xyz="0.0 0.068 0.0" />
+      <origin rpy="-1.57079633 -1.57079633 0" xyz="0.0 0.068 0.0" />
       <parent link="${prefix}b_and_r_cam"/>
       <child link="${prefix}tcp"/>

Commit message: dual arm setup - Not working yet

File: src/fmauch_universal_robot/ur_description/urdf/inc/b_and_r_cam_macro.xacro (robot description, xacro)
@@ -25,5 +25,5 @@
           use the "scale" param to compensate-->
           <mesh filename="package://ur_description/meshes/camera.stl"
-          scale="0.001 0.001 0.001"/>
+          scale="0.0012 0.0012 0.0012"/>
         </geometry>
         <material>

File: src/fmauch_universal_robot/ur_description/urdf/inc/b_and_r_light_bar_macro.xacro (robot description, xacro)
@@ -26,5 +26,5 @@
           use the "scale" param to compensate-->
           <mesh filename="package://ur_description/meshes/lightbar.stl"
-          scale="0.001 0.001 0.001"/>
+          scale="0.0012 0.0012 0.0012"/>
         </geometry>
         <material>

File: src/fmauch_universal_robot/ur_description/urdf/inc/mount_macro.xacro (robot description, xacro)
@@ -24,5 +24,5 @@
           <!-- The path to the collision meshes in the package. NOTE: mesh must be imported in metres, else
           use the "scale" param to compensate-->
-          <mesh filename="package://ur_description/meshes/mount.stl" scale="0.001 0.001 0.001" />
+          <mesh filename="package://ur_description/meshes/mount.stl" scale="0.0012 0.0012 0.0012" />
         </geometry>
         <material>
