Commit message: readme upd. + two robots tested IRL & working

File: src/group364_universal_robot/ur_description/urdf/inc/b_and_r_cam_macro.xacro (robot description, xacro)
@@ -25,5 +25,5 @@
           use the "scale" param to compensate-->
           <mesh filename="package://ur_description/meshes/camera.stl"
-          scale="0.0012 0.0012 0.0012"/>
+          scale="0.0013 0.0013 0.0013"/>
         </geometry>
         <material>

File: src/group364_universal_robot/ur_description/urdf/inc/b_and_r_light_bar_macro.xacro (robot description, xacro)
@@ -26,5 +26,5 @@
           use the "scale" param to compensate-->
           <mesh filename="package://ur_description/meshes/lightbar.stl"
-          scale="0.0012 0.0012 0.0012"/>
+          scale="0.0013 0.0013 0.0013"/>
         </geometry>
         <material>

File: src/group364_universal_robot/ur_description/urdf/inc/mount_macro.xacro (robot description, xacro)
@@ -24,5 +24,5 @@
           <!-- The path to the collision meshes in the package. NOTE: mesh must be imported in metres, else
           use the "scale" param to compensate-->
-          <mesh filename="package://ur_description/meshes/mount.stl" scale="0.0012 0.0012 0.0012" />
+          <mesh filename="package://ur_description/meshes/mount.stl" scale="0.0013 0.0013 0.0013" />
         </geometry>
         <material>

File: src/group364_universal_robot/ur_description/urdf/vision_application.xacro (robot description, xacro)
@@ -19,5 +19,5 @@
     <parent link="point_0" />
     <child link="ur5_light_bar_1_base_link" /> <!-- TODO: check base_link name of robot -->
-    <origin xyz="1.1945 0.176 -0.07" rpy="0.0 0.0 2.35619449" />
+    <origin xyz="1.1945 0.199 -0.07" rpy="0.0 0.0 2.35619449" />
   </joint>
 </robot>

Commit message: color on 3d mesh in rviz

File: src/group364_universal_robot/ur_description/urdf/inc/b_and_r_cam_macro.xacro (robot description, xacro)
@@ -19,4 +19,7 @@
           scale="0.001 0.001 0.001"/>
         </geometry>
+        <material name="b_and_r_color">
+          <color rgba="1 0.4 0 1"/>
+        </material>
       </visual>
       <collision>
@@ -27,6 +30,6 @@
           scale="0.0013 0.0013 0.0013"/>
         </geometry>
-        <material>
-          <color rgba="1 0.4 0 1"/>
+        <material name="collision">
+          <color rgba="0 0 1 1"/>
         </material>
       </collision>

File: src/group364_universal_robot/ur_description/urdf/inc/b_and_r_light_bar_macro.xacro (robot description, xacro)
@@ -20,4 +20,7 @@
           scale="0.001 0.001 0.001"/>
         </geometry>
+        <material name="b_and_r_color">
+          <color rgba="1 0.4 0 1"/>
+        </material>
       </visual>
       <collision>
@@ -28,6 +31,6 @@
           scale="0.0013 0.0013 0.0013"/>
         </geometry>
-        <material>
-          <color rgba="1 0.4 0"/>
+        <material name="collision">
+          <color rgba="0 0 1 1"/>
         </material>
       </collision>

File: src/group364_universal_robot/ur_description/urdf/inc/mount_macro.xacro (robot description, xacro)
@@ -19,4 +19,7 @@
           <mesh filename="package://ur_description/meshes/mount.stl" scale="0.001 0.001 0.001" />
         </geometry>
+        <material name="mount">
+          <color rgba="0.2 0.2 0.2 1" />
+        </material>
       </visual>
       <collision>
@@ -26,6 +29,6 @@
           <mesh filename="package://ur_description/meshes/mount.stl" scale="0.0013 0.0013 0.0013" />
         </geometry>
-        <material>
-          <color rgba="0 0 0 0" />
+        <material name="collision">
+          <color rgba="0 0 1 1"/>
         </material>
       </collision>

Commit message: extra padding on cam and light bar and wires

File: src/group364_universal_robot/ur_description/urdf/inc/b_and_r_cam_macro.xacro (robot description, xacro)
@@ -35,7 +35,41 @@
       </collision>
     </link>
+    <joint name="${prefix}wirecollisionbox_joint" type="fixed">
+      <origin rpy="0 0 0" xyz="0 -0.02 -0.03" />
+      <parent link="${prefix}b_and_r_cam"/>
+      <child link="${prefix}wirecollisionbox"/>
+    </joint>
+    <link name="${prefix}wirecollisionbox">
+      <visual>
+        <geometry>
+          <box size="0.09 0.02 0.09"/>
+        </geometry>
+      </visual>
+      <collision>
+        <geometry>
+          <box size="0.09 0.02 0.08"/>
+        </geometry>
+      </collision>
+    </link>
+    <joint name="${prefix}wirecollisionbox_2_joint" type="fixed">
+      <origin rpy="0 0 0" xyz="0 0.01 0.13" />
+      <parent link="${prefix}b_and_r_cam"/>
+      <child link="${prefix}wirecollisionbox_2"/>
+    </joint>
+    <link name="${prefix}wirecollisionbox_2">
+      <visual>
+        <geometry>
+          <box size="0.09 0.04 0.09"/>
+        </geometry>
+      </visual>
+      <collision>
+        <geometry>
+          <box size="0.09 0.04 0.09"/>
+        </geometry>
+      </collision>
+    </link>
     <!-- TCP frame -->
     <joint name="${prefix}tcp_joint" type="fixed">
-      <origin rpy="-1.57079633 -1.57079633 0" xyz="0.0 0.068 0.0" />
+      <origin rpy="-1.57079633 -1.57079633 0" xyz="0 0.062 -0.007" />
       <parent link="${prefix}b_and_r_cam"/>
       <child link="${prefix}tcp"/>

File: src/group364_universal_robot/ur_description/urdf/inc/b_and_r_light_bar_macro.xacro (robot description, xacro)
@@ -36,4 +36,21 @@
       </collision>
     </link>
+    <joint name="${prefix}wirecollisionbox_joint" type="fixed">
+      <origin rpy="0 0 0" xyz="0 -0.05 0" />
+      <parent link="${prefix}b_and_r_light_bar"/>
+      <child link="${prefix}wirecollisionbox"/>
+    </joint>
+    <link name="${prefix}wirecollisionbox">
+      <visual>
+        <geometry>
+          <box size="0.1 0.07 0.08"/>
+        </geometry>
+      </visual>
+      <collision>
+        <geometry>
+          <box size="0.1 0.07 0.08"/>
+        </geometry>
+      </collision>
+    </link>
     <!-- TCP frame -->
     <joint name="${prefix}tcp_joint" type="fixed">
